Commit message: Use xacros and pass in worldName
--HG--
branch : multicoptor

File: x1_description/urdf/x1_from_sdf.xacro (robot description, xacro)
@@ -1,5 +1,7 @@
 <?xml version='1.0' encoding='utf-8'?>
-<robot name='X1'>
-  <link name='tunnel_qual_ign/X1/base'>
+<robot name="X1" xmlns:xacro="http://ros.org/wiki/xacro">
+  <xacro:arg name="worldName" default=""/>
+  <xacro:property name="robot_namespace" value="$(arg worldName)/X1"/>
+  <link name='${robot_namespace}/base'>
     <inertial>
       <origin xyz='-0.00065 -0.085 0.062' rpy='0 -0 0'/>
@@ -123,65 +125,65 @@
   </link>
   <sensor name='imu_sensor' update_rate='1000'>
-    <parent link='tunnel_qual_ign/X1/base'/>
+    <parent link='${robot_namespace}/base'/>
     <origin xyz='0 0 0' rpy='0 -0 0'/>
   </sensor>
-  <link name='tunnel_qual_ign/X1/front_left_wheel'>
-    <inertial>
-      <origin xyz='0 0 0' rpy='0 -0 0'/>
-      <mass value='2.637'/>
-      <inertia ixx='0.02467' ixy='0' ixz='0' iyy='0.04411' iyz='0' izz='0.02467'/>
-    </inertial>
-    <collision name='collision'>
-      <origin xyz='0 0 0' rpy='-1.57079 0 0'/>
-      <geometry>
-        <cylinder radius='0.1651' length='0.1143'/>
-      </geometry>
-    </collision>
-    <visual name='visual'>
-      <origin xyz='0 0 0' rpy='0 -0 0'/>
-      <geometry>
-        <mesh filename='package://x1_description/meshes/wheel.dae' scale='1 1 1'/>
-      </geometry>
-    </visual>
-  </link>
-  <link name='tunnel_qual_ign/X1/front_right_wheel'>
-    <inertial>
-      <origin xyz='0 0 0' rpy='0 -0 0'/>
-      <mass value='2.637'/>
-      <inertia ixx='0.02467' ixy='0' ixz='0' iyy='0.04411' iyz='0' izz='0.02467'/>
-    </inertial>
-    <collision name='collision'>
-      <origin xyz='0 0 0' rpy='-1.57079 0 0'/>
-      <geometry>
-        <cylinder radius='0.1651' length='0.1143'/>
-      </geometry>
-    </collision>
-    <visual name='visual'>
-      <origin xyz='0 0 0' rpy='0 -0 0'/>
-      <geometry>
-        <mesh filename='package://x1_description/meshes/wheel.dae' scale='1 1 1'/>
-      </geometry>
-    </visual>
-  </link>
-  <link name='tunnel_qual_ign/X1/rear_left_wheel'>
-    <inertial>
-      <origin xyz='0 0 0' rpy='0 -0 0'/>
-      <mass value='2.637'/>
-      <inertia ixx='0.02467' ixy='0' ixz='0' iyy='0.04411' iyz='0' izz='0.02467'/>
-    </inertial>
-    <collision name='collision'>
-      <origin xyz='0 0 0' rpy='-1.57079 0 0'/>
-      <geometry>
-        <cylinder radius='0.1651' length='0.1143'/>
-      </geometry>
-    </collision>
-    <visual name='visual'>
-      <origin xyz='0 0 0' rpy='0 -0 0'/>
-      <geometry>
-        <mesh filename='package://x1_description/meshes/wheel.dae' scale='1 1 1'/>
-      </geometry>
-    </visual>
-  </link>
-  <link name='tunnel_qual_ign/X1/rear_right_wheel'>
+  <link name='${robot_namespace}/front_left_wheel'>
+    <inertial>
+      <origin xyz='0 0 0' rpy='0 -0 0'/>
+      <mass value='2.637'/>
+      <inertia ixx='0.02467' ixy='0' ixz='0' iyy='0.04411' iyz='0' izz='0.02467'/>
+    </inertial>
+    <collision name='collision'>
+      <origin xyz='0 0 0' rpy='-1.57079 0 0'/>
+      <geometry>
+        <cylinder radius='0.1651' length='0.1143'/>
+      </geometry>
+    </collision>
+    <visual name='visual'>
+      <origin xyz='0 0 0' rpy='0 -0 0'/>
+      <geometry>
+        <mesh filename='package://x1_description/meshes/wheel.dae' scale='1 1 1'/>
+      </geometry>
+    </visual>
+  </link>
+  <link name='${robot_namespace}/front_right_wheel'>
+    <inertial>
+      <origin xyz='0 0 0' rpy='0 -0 0'/>
+      <mass value='2.637'/>
+      <inertia ixx='0.02467' ixy='0' ixz='0' iyy='0.04411' iyz='0' izz='0.02467'/>
+    </inertial>
+    <collision name='collision'>
+      <origin xyz='0 0 0' rpy='-1.57079 0 0'/>
+      <geometry>
+        <cylinder radius='0.1651' length='0.1143'/>
+      </geometry>
+    </collision>
+    <visual name='visual'>
+      <origin xyz='0 0 0' rpy='0 -0 0'/>
+      <geometry>
+        <mesh filename='package://x1_description/meshes/wheel.dae' scale='1 1 1'/>
+      </geometry>
+    </visual>
+  </link>
+  <link name='${robot_namespace}/rear_left_wheel'>
+    <inertial>
+      <origin xyz='0 0 0' rpy='0 -0 0'/>
+      <mass value='2.637'/>
+      <inertia ixx='0.02467' ixy='0' ixz='0' iyy='0.04411' iyz='0' izz='0.02467'/>
+    </inertial>
+    <collision name='collision'>
+      <origin xyz='0 0 0' rpy='-1.57079 0 0'/>
+      <geometry>
+        <cylinder radius='0.1651' length='0.1143'/>
+      </geometry>
+    </collision>
+    <visual name='visual'>
+      <origin xyz='0 0 0' rpy='0 -0 0'/>
+      <geometry>
+        <mesh filename='package://x1_description/meshes/wheel.dae' scale='1 1 1'/>
+      </geometry>
+    </visual>
+  </link>
+  <link name='${robot_namespace}/rear_right_wheel'>
     <inertial>
       <origin xyz='0 0 0' rpy='0 -0 0'/>
@@ -204,6 +206,6 @@
   <joint name='front_left_wheel_joint' type='revolute'>
     <origin xyz='0.256 0.2854 0.03282' rpy='0 -0 0'/>
-    <parent link='tunnel_qual_ign/X1/base'/>
-    <child link='tunnel_qual_ign/X1/front_left_wheel'/>
+    <parent link='${robot_namespace}/base'/>
+    <child link='${robot_namespace}/front_left_wheel'/>
     <axis xyz='0 1 0'/>
     <limit lower='-1.79769e+308' upper='1.79769e+308' effort='-1' velocity='-1'/>
@@ -211,6 +213,6 @@
   <joint name='front_right_wheel_joint' type='revolute'>
     <origin xyz='0.256 -0.2854 0.03282' rpy='0 -0 0'/>
-    <parent link='tunnel_qual_ign/X1/base'/>
-    <child link='tunnel_qual_ign/X1/front_right_wheel'/>
+    <parent link='${robot_namespace}/base'/>
+    <child link='${robot_namespace}/front_right_wheel'/>
     <axis xyz='0 1 0'/>
     <limit lower='-1.79769e+308' upper='1.79769e+308' effort='-1' velocity='-1'/>
@@ -218,6 +220,6 @@
   <joint name='rear_left_wheel_joint' type='revolute'>
     <origin xyz='-0.256 0.2854 0.03282' rpy='0 -0 0'/>
-    <parent link='tunnel_qual_ign/X1/base'/>
-    <child link='tunnel_qual_ign/X1/rear_left_wheel'/>
+    <parent link='${robot_namespace}/base'/>
+    <child link='${robot_namespace}/rear_left_wheel'/>
     <axis xyz='0 1 0'/>
     <limit lower='-1.79769e+308' upper='1.79769e+308' effort='-1' velocity='-1'/>
@@ -225,6 +227,6 @@
   <joint name='rear_right_wheel_joint' type='revolute'>
     <origin xyz='-0.256 -0.2854 0.03282' rpy='0 -0 0'/>
-    <parent link='tunnel_qual_ign/X1/base'/>
-    <child link='tunnel_qual_ign/X1/rear_right_wheel'/>
+    <parent link='${robot_namespace}/base'/>
+    <child link='${robot_namespace}/rear_right_wheel'/>
     <axis xyz='0 1 0'/>
     <limit lower='-1.79769e+308' upper='1.79769e+308' effort='-1' velocity='-1'/>

File: x2_description/urdf/x2_from_sdf.xacro (robot description, xacro)
@@ -1,5 +1,7 @@
 <?xml version='1.0' encoding='utf-8'?>
-<robot name='X2'>
-  <link name='tunnel_qual_ign/X2/base'>
+<robot name="X2" xmlns:xacro="http://ros.org/wiki/xacro">
+  <xacro:arg name="worldName" default=""/>
+  <xacro:property name="robot_namespace" value="$(arg worldName)/X2"/>
+  <link name='${robot_namespace}/base'>
     <inertial>
       <origin xyz='0.011999 0.002 0.066996' rpy='0 -0 0'/>
@@ -51,8 +53,8 @@
   </link>
   <sensor name='imu_sensor' update_rate='1000'>
-    <parent link='tunnel_qual_ign/X2/base'/>
+    <parent link='${robot_namespace}/base'/>
     <origin xyz='0 0 0' rpy='0 -0 0'/>
   </sensor>
-  <link name='tunnel_qual_ign/X2/front_left_wheel'>
+  <link name='${robot_namespace}/front_left_wheel'>
     <inertial>
       <origin xyz='0 0 0' rpy='0 -0 0'/>
@@ -73,5 +75,5 @@
     </visual>
   </link>
-  <link name='tunnel_qual_ign/X2/front_right_wheel'>
+  <link name='${robot_namespace}/front_right_wheel'>
     <inertial>
       <origin xyz='0 0 0' rpy='0 -0 0'/>
@@ -92,5 +94,5 @@
     </visual>
   </link>
-  <link name='tunnel_qual_ign/X2/rear_left_wheel'>
+  <link name='${robot_namespace}/rear_left_wheel'>
     <inertial>
       <origin xyz='0 0 0' rpy='0 -0 0'/>
@@ -111,5 +113,5 @@
     </visual>
   </link>
-  <link name='tunnel_qual_ign/X2/rear_right_wheel'>
+  <link name='${robot_namespace}/rear_right_wheel'>
     <inertial>
       <origin xyz='0 0 0' rpy='0 -0 0'/>
@@ -132,6 +134,6 @@
   <joint name='front_left_wheel_joint' type='revolute'>
     <origin xyz='0.131 0.187795 0.0345' rpy='0 -0 0'/>
-    <parent link='tunnel_qual_ign/X2/base'/>
-    <child link='tunnel_qual_ign/X2/front_left_wheel'/>
+    <parent link='${robot_namespace}/base'/>
+    <child link='${robot_namespace}/front_left_wheel'/>
     <axis xyz='0 1 0'/>
     <limit lower='-1e+16' upper='1e+16' effort='-1' velocity='-1'/>
@@ -139,6 +141,6 @@
   <joint name='rear_left_wheel_joint' type='revolute'>
     <origin xyz='-0.131 0.187795 0.0345' rpy='0 -0 0'/>
-    <parent link='tunnel_qual_ign/X2/base'/>
-    <child link='tunnel_qual_ign/X2/rear_left_wheel'/>
+    <parent link='${robot_namespace}/base'/>
+    <child link='${robot_namespace}/rear_left_wheel'/>
     <axis xyz='0 1 0'/>
     <limit lower='-1.79769e+308' upper='1.79769e+308' effort='-1' velocity='-1'/>
@@ -146,6 +148,6 @@
   <joint name='rear_right_wheel_joint' type='revolute'>
     <origin xyz='-0.131 -0.187795 0.0345' rpy='0 -0 0'/>
-    <parent link='tunnel_qual_ign/X2/base'/>
-    <child link='tunnel_qual_ign/X2/rear_right_wheel'/>
+    <parent link='${robot_namespace}/base'/>
+    <child link='${robot_namespace}/rear_right_wheel'/>
     <axis xyz='0 1 0'/>
     <limit lower='-1.79769e+308' upper='1.79769e+308' effort='-1' velocity='-1'/>
@@ -153,6 +155,6 @@
   <joint name='front_right_wheel_joint' type='revolute'>
     <origin xyz='0.131 -0.187795 0.0345' rpy='0 -0 0'/>
-    <parent link='tunnel_qual_ign/X2/base'/>
-    <child link='tunnel_qual_ign/X2/front_right_wheel'/>
+    <parent link='${robot_namespace}/base'/>
+    <child link='${robot_namespace}/front_right_wheel'/>
     <axis xyz='0 1 0'/>
     <limit lower='-1.79769e+308' upper='1.79769e+308' effort='-1' velocity='-1'/>

File: x3_description/urdf/x3_from_sdf.xacro (robot description, xacro)
@@ -1,5 +1,7 @@
 <?xml version='1.0' encoding='utf-8'?>
-<robot name='X3'>
-  <link name='tunnel_qual_ign/X3/base_link'>
+<robot name="X3" xmlns:xacro="http://ros.org/wiki/xacro">
+  <xacro:arg name="worldName" default=""/>
+  <xacro:property name="robot_namespace" value="$(arg worldName)/X3"/>
+  <link name='${robot_namespace}/base_link'>
     <inertial>
       <origin xyz='0 0 0' rpy='0 -0 0'/>
@@ -21,8 +23,8 @@
   </link>
   <sensor name='imu_sensor' update_rate='1000'>
-    <parent link='tunnel_qual_ign/X3/base_link'/>
+    <parent link='${robot_namespace}/base_link'/>
     <origin xyz='0 0 0' rpy='0 -0 0'/>
   </sensor>
-  <link name='tunnel_qual_ign/X3/rotor_0'>
+  <link name='${robot_namespace}/rotor_0'>
     <inertial>
       <origin xyz='0 0 0' rpy='0 -0 0'/>
@@ -43,5 +45,5 @@
     </visual>
   </link>
-  <link name='tunnel_qual_ign/X3/rotor_1'>
+  <link name='${robot_namespace}/rotor_1'>
     <inertial>
       <origin xyz='0 0 0' rpy='0 -0 0'/>
@@ -62,5 +64,5 @@
     </visual>
   </link>
-  <link name='tunnel_qual_ign/X3/rotor_2'>
+  <link name='${robot_namespace}/rotor_2'>
     <inertial>
       <origin xyz='0 0 0' rpy='0 -0 0'/>
@@ -81,5 +83,5 @@
     </visual>
   </link>
-  <link name='tunnel_qual_ign/X3/rotor_3'>
+  <link name='${robot_namespace}/rotor_3'>
     <inertial>
       <origin xyz='0 0 0' rpy='0 -0 0'/>
@@ -102,6 +104,6 @@
   <joint name='rotor_0_joint' type='revolute'>
     <origin xyz='0.13 -0.22 0.023' rpy='0 -0 0'/>
-    <parent link='tunnel_qual_ign/X3/base_link'/>
-    <child link='tunnel_qual_ign/X3/rotor_0'/>
+    <parent link='${robot_namespace}/base_link'/>
+    <child link='${robot_namespace}/rotor_0'/>
     <dynamics damping='0' friction='0' />
     <axis xyz='0 0 1'/>
@@ -110,6 +112,6 @@
   <joint name='rotor_1_joint' type='revolute'>
     <origin xyz='-0.13 0.2 0.023' rpy='0 -0 0'/>
-    <parent link='tunnel_qual_ign/X3/base_link'/>
-    <child link='tunnel_qual_ign/X3/rotor_1'/>
+    <parent link='${robot_namespace}/base_link'/>
+    <child link='${robot_namespace}/rotor_1'/>
     <dynamics damping='0' friction='0' />
     <axis xyz='0 0 1'/>
@@ -118,6 +120,6 @@
   <joint name='rotor_2_joint' type='revolute'>
     <origin xyz='0.13 0.22 0.023' rpy='0 -0 0'/>
-    <parent link='tunnel_qual_ign/X3/base_link'/>
-    <child link='tunnel_qual_ign/X3/rotor_2'/>
+    <parent link='${robot_namespace}/base_link'/>
+    <child link='${robot_namespace}/rotor_2'/>
     <dynamics damping='0' friction='0' />
     <axis xyz='0 0 1'/>
@@ -126,6 +128,6 @@
   <joint name='rotor_3_joint' type='revolute'>
     <origin xyz='-0.13 -0.2 0.023' rpy='0 -0 0'/>
-    <parent link='tunnel_qual_ign/X3/base_link'/>
-    <child link='tunnel_qual_ign/X3/rotor_3'/>
+    <parent link='${robot_namespace}/base_link'/>
+    <child link='${robot_namespace}/rotor_3'/>
     <dynamics damping='0' friction='0' />
     <axis xyz='0 0 1'/>

File: x4_description/urdf/x4_from_sdf.xacro (robot description, xacro)
@@ -1,5 +1,7 @@
 <?xml version='1.0' encoding='utf-8'?>
-<robot name='X4'>
-  <link name='tunnel_qual_ign/X4/base_link'>
+<robot name="X4" xmlns:xacro="http://ros.org/wiki/xacro">
+  <xacro:arg name="worldName" default=""/>
+  <xacro:property name="robot_namespace" value="$(arg worldName)/X4"/>
+  <link name='${robot_namespace}/base_link'>
     <inertial>
       <origin xyz='0 0 0' rpy='0 -0 0'/>
@@ -21,8 +23,8 @@
   </link>
   <sensor name='imu_sensor' update_rate='1000'>
-    <parent link='tunnel_qual_ign/X4/base_link'/>
+    <parent link='${robot_namespace}/base_link'/>
     <origin xyz='0 0 0' rpy='0 -0 0'/>
   </sensor>
-  <link name='tunnel_qual_ign/X4/rotor_0'>
+  <link name='${robot_namespace}/rotor_0'>
     <inertial>
       <origin xyz='0 0 0' rpy='0 -0 0'/>
@@ -43,5 +45,5 @@
     </visual>
   </link>
-  <link name='tunnel_qual_ign/X4/rotor_1'>
+  <link name='${robot_namespace}/rotor_1'>
     <inertial>
       <origin xyz='0 0 0' rpy='0 -0 0'/>
@@ -62,5 +64,5 @@
     </visual>
   </link>
-  <link name='tunnel_qual_ign/X4/rotor_2'>
+  <link name='${robot_namespace}/rotor_2'>
     <inertial>
       <origin xyz='0 0 0' rpy='0 -0 0'/>
@@ -81,5 +83,5 @@
     </visual>
   </link>
-  <link name='tunnel_qual_ign/X4/rotor_3'>
+  <link name='${robot_namespace}/rotor_3'>
     <inertial>
       <origin xyz='0 0 0' rpy='0 -0 0'/>
@@ -100,5 +102,5 @@
     </visual>
   </link>
-  <link name='tunnel_qual_ign/X4/rotor_4'>
+  <link name='${robot_namespace}/rotor_4'>
     <inertial>
       <origin xyz='0 0 0' rpy='-0 -0 -0'/>
@@ -119,5 +121,5 @@
     </visual>
   </link>
-  <link name='tunnel_qual_ign/X4/rotor_5'>
+  <link name='${robot_namespace}/rotor_5'>
     <inertial>
       <origin xyz='0 0 0' rpy='0 -0 0'/>
@@ -140,6 +142,6 @@
   <joint name='rotor_0_joint' type='revolute'>
     <origin xyz='0.247 0.1506 0.028' rpy='0.087267 0 0.523599'/>
-    <parent link='tunnel_qual_ign/X4/base_link'/>
-    <child link='tunnel_qual_ign/X4/rotor_0'/>
+    <parent link='${robot_namespace}/base_link'/>
+    <child link='${robot_namespace}/rotor_0'/>
     <dynamics damping='0' friction='0' />
     <axis xyz='0 1e-06 1'/>
@@ -148,6 +150,6 @@
   <joint name='rotor_1_joint' type='revolute'>
     <origin xyz='-0.00067 0.28929 0.028' rpy='0 -0.087267 0'/>
-    <parent link='tunnel_qual_ign/X4/base_link'/>
-    <child link='tunnel_qual_ign/X4/rotor_1'/>
+    <parent link='${robot_namespace}/base_link'/>
+    <child link='${robot_namespace}/rotor_1'/>
     <dynamics damping='0' friction='0' />
     <axis xyz='0 0 1'/>
@@ -156,6 +158,6 @@
   <joint name='rotor_2_joint' type='revolute'>
     <origin xyz='-0.2501 0.1454 0.028' rpy='0.087267 -0 2.61799'/>
-    <parent link='tunnel_qual_ign/X4/base_link'/>
-    <child link='tunnel_qual_ign/X4/rotor_2'/>
+    <parent link='${robot_namespace}/base_link'/>
+    <child link='${robot_namespace}/rotor_2'/>
     <dynamics damping='0' friction='0' />
     <axis xyz='0 1e-06 1'/>
@@ -164,6 +166,6 @@
   <joint name='rotor_3_joint' type='revolute'>
     <origin xyz='-0.2501 -0.1454 0.028' rpy='-0.087267 -0 -2.61799'/>
-    <parent link='tunnel_qual_ign/X4/base_link'/>
-    <child link='tunnel_qual_ign/X4/rotor_3'/>
+    <parent link='${robot_namespace}/base_link'/>
+    <child link='${robot_namespace}/rotor_3'/>
     <dynamics damping='0' friction='0' />
     <axis xyz='0 -1e-06 1'/>
@@ -172,6 +174,6 @@
   <joint name='rotor_4_joint' type='revolute'>
     <origin xyz='-0.00067 -0.28929 0.028' rpy='-0 0.087267 -3.14159'/>
-    <parent link='tunnel_qual_ign/X4/base_link'/>
-    <child link='tunnel_qual_ign/X4/rotor_4'/>
+    <parent link='${robot_namespace}/base_link'/>
+    <child link='${robot_namespace}/rotor_4'/>
     <dynamics damping='0' friction='0' />
     <axis xyz='-0 -0 1'/>
@@ -180,6 +182,6 @@
   <joint name='rotor_5_joint' type='revolute'>
     <origin xyz='0.247 -0.1506 0.028' rpy='-0.087267 0 -0.523599'/>
-    <parent link='tunnel_qual_ign/X4/base_link'/>
-    <child link='tunnel_qual_ign/X4/rotor_5'/>
+    <parent link='${robot_namespace}/base_link'/>
+    <child link='${robot_namespace}/rotor_5'/>
     <dynamics damping='0' friction='0' />
     <axis xyz='0 -1e-06 1'/>

Commit message: ROS integration for virtual_stix
--HG--
branch : virtual_stix_ros

File: x1_description/urdf/x1_from_sdf.xacro (robot description, xacro)
@@ -1,6 +1,6 @@
 <?xml version='1.0' encoding='utf-8'?>
 <robot name="X1" xmlns:xacro="http://ros.org/wiki/xacro">
-  <xacro:arg name="worldName" default=""/>
-  <xacro:property name="robot_namespace" value="$(arg worldName)/X1"/>
+  <xacro:arg name="world_name" default=""/>
+  <xacro:property name="robot_namespace" value="$(arg world_name)/X1"/>
   <link name='${robot_namespace}/base'>
     <inertial>

File: x2_description/urdf/x2_from_sdf.xacro (robot description, xacro)
@@ -1,6 +1,6 @@
 <?xml version='1.0' encoding='utf-8'?>
 <robot name="X2" xmlns:xacro="http://ros.org/wiki/xacro">
-  <xacro:arg name="worldName" default=""/>
-  <xacro:property name="robot_namespace" value="$(arg worldName)/X2"/>
+  <xacro:arg name="world_name" default=""/>
+  <xacro:property name="robot_namespace" value="$(arg world_name)/X2"/>
   <link name='${robot_namespace}/base'>
     <inertial>

File: x3_description/urdf/x3_from_sdf.xacro (robot description, xacro)
@@ -1,6 +1,6 @@
 <?xml version='1.0' encoding='utf-8'?>
 <robot name="X3" xmlns:xacro="http://ros.org/wiki/xacro">
-  <xacro:arg name="worldName" default=""/>
-  <xacro:property name="robot_namespace" value="$(arg worldName)/X3"/>
+  <xacro:arg name="world_name" default=""/>
+  <xacro:property name="robot_namespace" value="$(arg world_name)/X3"/>
   <link name='${robot_namespace}/base_link'>
     <inertial>

File: x4_description/urdf/x4_from_sdf.xacro (robot description, xacro)
@@ -1,6 +1,6 @@
 <?xml version='1.0' encoding='utf-8'?>
 <robot name="X4" xmlns:xacro="http://ros.org/wiki/xacro">
-  <xacro:arg name="worldName" default=""/>
-  <xacro:property name="robot_namespace" value="$(arg worldName)/X4"/>
+  <xacro:arg name="world_name" default=""/>
+  <xacro:property name="robot_namespace" value="$(arg world_name)/X4"/>
   <link name='${robot_namespace}/base_link'>
     <inertial>
