Commit message: Modify topic remaps to use sensor default topics
--HG--
branch : remap_default_topics

File: x1_description/urdf/x1_from_sdf.xacro (robot description, xacro)
@@ -1,7 +1,7 @@
 <?xml version='1.0' encoding='utf-8'?>
 <robot name="X1" xmlns:xacro="http://ros.org/wiki/xacro">
-  <xacro:arg name="world_name" default=""/>
-  <xacro:property name="robot_namespace" value="$(arg world_name)/X1"/>
-  <link name='${robot_namespace}/base'>
+  <xacro:arg name="name" default="X1"/>
+  <xacro:property name="robot_namespace" value="$(arg name)"/>
+  <link name='${robot_namespace}/base_link'>
     <inertial>
       <origin xyz='-0.00065 -0.085 0.062' rpy='0 -0 0'/>
@@ -125,5 +125,5 @@
   </link>
   <sensor name='imu_sensor' update_rate='1000'>
-    <parent link='${robot_namespace}/base'/>
+    <parent link='${robot_namespace}/base_link'/>
     <origin xyz='0 0 0' rpy='0 -0 0'/>
   </sensor>
@@ -206,5 +206,5 @@
   <joint name='front_left_wheel_joint' type='revolute'>
     <origin xyz='0.256 0.2854 0.03282' rpy='0 -0 0'/>
-    <parent link='${robot_namespace}/base'/>
+    <parent link='${robot_namespace}/base_link'/>
     <child link='${robot_namespace}/front_left_wheel'/>
     <axis xyz='0 1 0'/>
@@ -213,5 +213,5 @@
   <joint name='front_right_wheel_joint' type='revolute'>
     <origin xyz='0.256 -0.2854 0.03282' rpy='0 -0 0'/>
-    <parent link='${robot_namespace}/base'/>
+    <parent link='${robot_namespace}/base_link'/>
     <child link='${robot_namespace}/front_right_wheel'/>
     <axis xyz='0 1 0'/>
@@ -220,5 +220,5 @@
   <joint name='rear_left_wheel_joint' type='revolute'>
     <origin xyz='-0.256 0.2854 0.03282' rpy='0 -0 0'/>
-    <parent link='${robot_namespace}/base'/>
+    <parent link='${robot_namespace}/base_link'/>
     <child link='${robot_namespace}/rear_left_wheel'/>
     <axis xyz='0 1 0'/>
@@ -227,5 +227,5 @@
   <joint name='rear_right_wheel_joint' type='revolute'>
     <origin xyz='-0.256 -0.2854 0.03282' rpy='0 -0 0'/>
-    <parent link='${robot_namespace}/base'/>
+    <parent link='${robot_namespace}/base_link'/>
     <child link='${robot_namespace}/rear_right_wheel'/>
     <axis xyz='0 1 0'/>

File: x2_description/urdf/x2_from_sdf.xacro (robot description, xacro)
@@ -1,7 +1,7 @@
 <?xml version='1.0' encoding='utf-8'?>
 <robot name="X2" xmlns:xacro="http://ros.org/wiki/xacro">
-  <xacro:arg name="world_name" default=""/>
-  <xacro:property name="robot_namespace" value="$(arg world_name)/X2"/>
-  <link name='${robot_namespace}/base'>
+  <xacro:arg name="name" default="X2"/>
+  <xacro:property name="robot_namespace" value="$(arg name)"/>
+  <link name='${robot_namespace}/base_link'>
     <inertial>
       <origin xyz='0.011999 0.002 0.066996' rpy='0 -0 0'/>
@@ -53,5 +53,5 @@
   </link>
   <sensor name='imu_sensor' update_rate='1000'>
-    <parent link='${robot_namespace}/base'/>
+    <parent link='${robot_namespace}/base_link'/>
     <origin xyz='0 0 0' rpy='0 -0 0'/>
   </sensor>
@@ -134,5 +134,5 @@
   <joint name='front_left_wheel_joint' type='revolute'>
     <origin xyz='0.131 0.187795 0.0345' rpy='0 -0 0'/>
-    <parent link='${robot_namespace}/base'/>
+    <parent link='${robot_namespace}/base_link'/>
     <child link='${robot_namespace}/front_left_wheel'/>
     <axis xyz='0 1 0'/>
@@ -141,5 +141,5 @@
   <joint name='rear_left_wheel_joint' type='revolute'>
     <origin xyz='-0.131 0.187795 0.0345' rpy='0 -0 0'/>
-    <parent link='${robot_namespace}/base'/>
+    <parent link='${robot_namespace}/base_link'/>
     <child link='${robot_namespace}/rear_left_wheel'/>
     <axis xyz='0 1 0'/>
@@ -148,5 +148,5 @@
   <joint name='rear_right_wheel_joint' type='revolute'>
     <origin xyz='-0.131 -0.187795 0.0345' rpy='0 -0 0'/>
-    <parent link='${robot_namespace}/base'/>
+    <parent link='${robot_namespace}/base_link'/>
     <child link='${robot_namespace}/rear_right_wheel'/>
     <axis xyz='0 1 0'/>
@@ -155,5 +155,5 @@
   <joint name='front_right_wheel_joint' type='revolute'>
     <origin xyz='0.131 -0.187795 0.0345' rpy='0 -0 0'/>
-    <parent link='${robot_namespace}/base'/>
+    <parent link='${robot_namespace}/base_link'/>
     <child link='${robot_namespace}/front_right_wheel'/>
     <axis xyz='0 1 0'/>

File: x3_description/urdf/x3_from_sdf.xacro (robot description, xacro)
@@ -1,6 +1,6 @@
 <?xml version='1.0' encoding='utf-8'?>
 <robot name="X3" xmlns:xacro="http://ros.org/wiki/xacro">
-  <xacro:arg name="world_name" default=""/>
-  <xacro:property name="robot_namespace" value="$(arg world_name)/X3"/>
+  <xacro:arg name="name" default="X3"/>
+  <xacro:property name="robot_namespace" value="$(arg name)"/>
   <link name='${robot_namespace}/base_link'>
     <inertial>

File: x4_description/urdf/x4_from_sdf.xacro (robot description, xacro)
@@ -1,6 +1,6 @@
 <?xml version='1.0' encoding='utf-8'?>
 <robot name="X4" xmlns:xacro="http://ros.org/wiki/xacro">
-  <xacro:arg name="world_name" default=""/>
-  <xacro:property name="robot_namespace" value="$(arg world_name)/X4"/>
+  <xacro:arg name="name" default="X4"/>
+  <xacro:property name="robot_namespace" value="$(arg name)"/>
   <link name='${robot_namespace}/base_link'>
     <inertial>
